File: hardware/BMP_Bluepill.kicad_sch (KiCad schematic)
At the start: 30 parts, among them J1 Conn_01x06, J2 USB_C_Receptacle_USB2.0_16P, J3 Conn_01x04, U1 STM32F103C8T6, U2 AMS1117-3.3, Y1 8 MHz

Commit message: update layout
Parts:
- removed D3: LED, LED_SMD:LED_0603_1608Metric_Pad1.05x0.95mm_HandSolder, symbol Device:LED
- removed R5: 10k[N/A], Resistor_SMD:R_0603_1608Metric_Pad0.98x0.95mm_HandSolder, symbol Device:R
- removed R6: 1k, Resistor_SMD:R_0603_1608Metric_Pad0.98x0.95mm_HandSolder, symbol Device:R
- removed Y1: 8 MHz, Crystal:Crystal_HC49-4H_Vertical, symbol Device:Crystal
- added Y2: 8MHz, Crystal:Crystal_SMD_5032-4Pin_5.0x3.2mm, symbol Device:Crystal_GND24
Connections:
- net +3V3: now also D2.2 (A), U2.4 (EPAD)
- net GND: now also J2.S1 (SHIELD), Y2.2, Y2.4; no longer D2.1 (K)
- net at R4.2: now also D2.1 (K); no longer D2.2 (A)
- net at C13.1, U1.5 (OSC_IN): now also Y2.1
- net at C14.1, U1.6 (OSC_OUT): now also Y2.3
- net LED_UART: no longer names the net of U1.30 (PA9)
- no-connect marks 5 -> 27
Other:
- moved on the sheet: D1, D2, R2, R3, R4
